Commit message: Add files via upload

File: hb_task_1b/urdf/hb_bot.urdf.xacro (robot description, xacro)
@@ -9,7 +9,7 @@
 *
 *  Filename:            hb_bot.urdf.xacro
-*  Created:             08th october 2023
+*  Created:             10th october 2023
 *  Last Modified:
-*  Author:              Raj Aryan
+*  Author:             Raj Aryan
 *
 *****************************************************************************************
@@ -18,10 +18,6 @@
 <!-- Start of Robot Definition
 Inside which we shall have all of the remaining definitions, which will end with the last line of the file: -->
-     <xacro:include filename="$(find holo)/urdf/materials.xacro"/>
-    <!-- material properties of right wheel -->
-    <gazebo reference="right_wheel">
-        <material>Gazebo/Black</material>
-    </gazebo>
-    <!-- base link -->
+    <xacro:include filename="$(find holo)/urdf/materials.xacro"/>
+    <!--Base link-->
     <link name ="base_link">
         <inertial>
@@ -55,108 +51,7 @@
         </visual>
     </link>
-    <!-- footprint link -->
     <link name ="footprint_link">
         <!-- empty link -->
     </link>
-    <!-- front_wheel -->
-    <link name ="front_wheel">
-        <inertial>
-            <origin
-                xyz="0 -0.05 0.0"
-                rpy="1.57 0 0" />
-            <mass
-                value="0.060" />
-            <inertia
-                ixx="1.825e-4"
-                ixy="0"
-                ixz="0.00000000"
-                iyy="1.825e-4"
-                iyz="0"
-                izz="1.825e-4" />
-        </inertial>
-        <collision name="F_collision">
-         <origin
-                xyz="0 -0.05 0.0"
-                rpy="1.57 0 0" />
-          <geometry>
-            <cylinder length="0.13" radius="0.14"/>
-          </geometry>
-        </collision>
-        <visual>
-            <origin
-            xyz="0.0 0.0 0.0"
-            rpy="0.0 0.0 0.0" />
-            <geometry>
-                <mesh filename ="file://$(find holo)/meshes/wheel.stl" scale="5 5 5"/>
-            </geometry>
-        </visual>
-    </link>
-    <!-- left wheel -->
-    <link name ="left_wheel">
-        <inertial>
-            <origin
-                xyz="0.15154 0.087275 0.0"
-                rpy="1.57 0 0" />
-            <mass
-                value="0.060" />
-            <inertia
-                ixx="1.825e-4"
-                ixy="0"
-                ixz="0.00000000"
-                iyy="1.825e-4"
-                iyz="0"
-                izz="1.825e-4" />
-        </inertial>
-        <collision name="L_collision">
-         <origin
-                xyz="0.15154 0.087275 0.0"
-                rpy="1.57 0 0" />
-          <geometry>
-            <cylinder length="0.13" radius="0.14"/>
-          </geometry>
-        </collision>
-        <visual>
-            <origin
-            xyz="0.15154 0.087275 0.0"
-            rpy="0.0 0.0 0.0" />
-            <geometry>
-                <mesh filename ="file://$(find holo)/meshes/wheel.stl" scale="5 5 5"/>
-            </geometry>
-        </visual>
-    </link>
-    <!-- right_wheel -->
-    <link name ="right_wheel">
-        <inertial>
-            <origin
-                xyz="-0.15154 -0.087275 0.0"
-                rpy="1.57 0 0" />
-            <mass
-                value="0.060" />
-            <inertia
-                ixx="1.825e-4"
-                ixy="0"
-                ixz="0.00000000"
-                iyy="1.825e-4"
-                iyz="0"
-                izz="1.825e-4" />
-        </inertial>
-        <collision name="R_collision">
-         <origin
-                xyz="-0.15154 -0.087275 0.0"
-                rpy="1.57 0 0" />
-          <geometry>
-            <cylinder length="0.13" radius="0.14"/>
-          </geometry>
-        </collision>
-        <visual>
-            <origin
-            xyz="-0.15154 -0.087275 0.0"
-            rpy="0.0 0.0 0.0" />
-            <geometry>
-                <mesh filename ="file://$(find holo)/meshes/wheel.stl" scale="5 5 5"/>
-            </geometry>
-        </visual>
-    </link>
-    <!-- joint between footprint_link and base_link -->
     <joint name="footprint_joint" type="fixed">
          <origin
@@ -166,49 +61,3 @@
         <child link="base_link"/>
     </joint>
-    <!-- joint between base_link and front_wheel -->
-    <joint name ="front_wheel_joint" type="continuous" >
-        <origin
-                xyz="0.0 0.68 0.18"
-                rpy="0 0 0" />
-        <parent link="base_link"/>
-        <child link="right_wheel"/>
-        <axis xyz="0.0 1.0 0.0"/>
-         <limit
-            effort="5"
-            velocity="5" />
-    </joint>
-    <!-- joint between base_link and left_wheel -->
-    <joint name ="left_wheel_joint" type="continuous" >
-        <origin
-                xyz="0.15154 0.087275 0.18"
-                rpy="0 0 0" />
-        <parent link="base_link"/>
-        <child link="right_wheel"/>
-        <axis xyz="0.0 1.0 0.0"/>
-         <limit
-            effort="5"
-            velocity="5" />
-    </joint>
-    <!-- joint between base_link and right_wheel -->
-    <joint name ="right_wheel_joint" type="continuous" >
-        <origin
-                xyz="-0.15154 -0.08725 0.18"
-                rpy="0 0 0" />
-        <parent link="base_link"/>
-        <child link="right_wheel"/>
-        <axis xyz="0.0 1.0 0.0"/>
-         <limit
-            effort="5"
-            velocity="5" />
-    </joint>
-    <!-- ros_control plugin -->
-  <gazebo>
-    <plugin name="object_controller" filename="libgazebo_ros_planar_move.so">
-      <commandTopic>cmd_vel</commandTopic>
-      <odometryTopic>odom</odometryTopic>
-      <odometryFrame>odom</odometryFrame>
-      <odometryRate>20.0</odometryRate>
-      <robotBaseFrame>chasis</robotBaseFrame>
-    </plugin>
-  </gazebo>
 </robot>
